File: Hardware/Xbee_shield.sch (EAGLE design)
At the start: 37 parts, among them Q1 MOSFET-NCHANNELSMD, Q2 MOSFET-NCHANNELSMD, U1 ARDUINO_SHIELD, U2 XBEE-1B3, U4 V_REG_LDOSMD

Commit message: Changes to Silk/SCH
Parts:
- JP4: value (none) -> M10"; device SparkFun:M06SIP -> SparkFun-Connectors:M10"
Connections:
- removed net N$67: JP4.6, U1.D13, U1.SCL, U1.SDA
- new net AREF: JP4.8, U1.AREF
- new net N$3: JP4.6, U1.D13
- new net N$6: JP4.9, U1.SDA
- new net N$7: JP4.10, U1.SCL
- net GND: now also JP4.7
Other:
- moved on the sheet: JP1
Changed lines of the file:
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@@
 <setting verticaltext="up"/>
 </settings>
-<grid distance="0.1" unitdist="inch" unit="inch" style="lines" multiple="1" display="no" altdistance="0.01" altunitdist="inch" altunit="inch"/>
+<grid distance="0.1" unitdist="inch" unit="inch" style="lines" multiple="1" display="no" altdistance="0.001" altunitdist="inch" altunit="inch"/>
 <layers>
 <layer number="1" name="Top" color="4" fill="1" visible="no" active="no"/>
@@
 <part name="SJ3" library="SparkFun" deviceset="SOLDERJUMPER" device="NC" value="D_RX"/>
 <part name="JP1" library="SparkFun" deviceset="M06" device="SIP"/>
-<part name="JP4" library="SparkFun" deviceset="M06" device="SIP"/>
+<part name="JP4" library="SparkFun-Connectors" deviceset="M10" device="&quot;" value=""/>
 <part name="JP5" library="SparkFun" deviceset="FIDUCIAL" device="1X2"/>
 <part name="JP6" library="SparkFun" deviceset="FIDUCIAL" device="1X2"/>
@@
 <part name="U$9" library="SparkFun" deviceset="5V" device=""/>
 <part name="JP7" library="SparkFun-Aesthetics" deviceset="LOGO-SFE" device="NEW"/>
+<part name="GND10" library="SparkFun" deviceset="GND" device=""/>
 </parts>
 <sheets>
@@
 <instance part="SJ1" gate="1" x="127" y="154.94" rot="R90"/>
 <instance part="SJ3" gate="1" x="137.16" y="154.94" rot="R90"/>
-<instance part="JP1" gate="G$1" x="83.82" y="111.76" rot="R180"/>
-<instance part="JP4" gate="G$1" x="83.82" y="88.9" rot="R180"/>
+<instance part="JP1" gate="G$1" x="101.6" y="111.76" rot="R180"/>
+<instance part="JP4" gate="G$1" x="106.68" y="76.2" rot="R180"/>
 <instance part="JP5" gate="G$1" x="243.84" y="38.1"/>
 <instance part="JP6" gate="G$1" x="238.76" y="38.1"/>
@@
 <instance part="U$9" gate="G$1" x="205.74" y="121.92"/>
 <instance part="JP7" gate="G$1" x="231.14" y="17.78"/>
+<instance part="GND10" gate="1" x="93.98" y="66.04"/>
 </instances>
 <busses>
@@
 <pinref part="GND9" gate="1" pin="GND"/>
 </segment>
+<segment>
+<pinref part="JP4" gate="G$1" pin="7"/>
+<wire x1="96.52" y1="78.74" x2="93.98" y2="78.74" width="0.1524" layer="91"/>
+<wire x1="93.98" y1="78.74" x2="93.98" y2="68.58" width="0.1524" layer="91"/>
+<pinref part="GND10" gate="1" pin="GND"/>
+</segment>
 </net>
 <net name="RESET" class="0">
@@
 <net name="D_TX" class="0">
 <segment>
-<wire x1="66.04" y1="114.3" x2="78.74" y2="114.3" width="0.1524" layer="91"/>
+<wire x1="66.04" y1="114.3" x2="96.52" y2="114.3" width="0.1524" layer="91"/>
 <label x="68.58" y="114.3" size="1.778" layer="95"/>
 <pinref part="U1" gate="G$1" pin="*D3"/>
@@
 <net name="D_RX" class="0">
 <segment>
-<wire x1="66.04" y1="116.84" x2="78.74" y2="116.84" width="0.1524" layer="91"/>
+<wire x1="66.04" y1="116.84" x2="96.52" y2="116.84" width="0.1524" layer="91"/>
 <label x="68.58" y="116.84" size="1.778" layer="95"/>
 <pinref part="U1" gate="G$1" pin="D2"/>
@@
 <net name="N$142" class="0">
 <segment>
-<wire x1="66.04" y1="111.76" x2="78.74" y2="111.76" width="0.1524" layer="91"/>
+<wire x1="66.04" y1="111.76" x2="96.52" y2="111.76" width="0.1524" layer="91"/>
 <pinref part="U1" gate="G$1" pin="D4"/>
 <pinref part="JP1" gate="G$1" pin="3"/>
@@
 <net name="N$143" class="0">
 <segment>
-<wire x1="66.04" y1="109.22" x2="78.74" y2="109.22" width="0.1524" layer="91"/>
+<wire x1="66.04" y1="109.22" x2="96.52" y2="109.22" width="0.1524" layer="91"/>
 <pinref part="U1" gate="G$1" pin="*D5"/>
 <pinref part="JP1" gate="G$1" pin="4"/>
@@
 <net name="N$144" class="0">
 <segment>
-<wire x1="66.04" y1="106.68" x2="78.74" y2="106.68" width="0.1524" layer="91"/>
+<wire x1="66.04" y1="106.68" x2="96.52" y2="106.68" width="0.1524" layer="91"/>
 <pinref part="U1" gate="G$1" pin="*D6"/>
 <pinref part="JP1" gate="G$1" pin="5"/>
@@
 <net name="N$145" class="0">
 <segment>
-<wire x1="66.04" y1="104.14" x2="78.74" y2="104.14" width="0.1524" layer="91"/>
+<wire x1="66.04" y1="104.14" x2="96.52" y2="104.14" width="0.1524" layer="91"/>
 <pinref part="U1" gate="G$1" pin="D7"/>
 <pinref part="JP1" gate="G$1" pin="6"/>
@@
 <net name="N$17" class="0">
 <segment>
-<wire x1="66.04" y1="101.6" x2="78.74" y2="101.6" width="0.1524" layer="91"/>
-<wire x1="78.74" y1="101.6" x2="78.74" y2="93.98" width="0.1524" layer="91"/>
+<wire x1="66.04" y1="101.6" x2="88.9" y2="101.6" width="0.1524" layer="91"/>
 <pinref part="U1" gate="G$1" pin="D8"/>
 <pinref part="JP4" gate="G$1" pin="1"/>
+<wire x1="96.52" y1="93.98" x2="88.9" y2="93.98" width="0.1524" layer="91"/>
+<wire x1="88.9" y1="93.98" x2="88.9" y2="101.6" width="0.1524" layer="91"/>
 </segment>
 </net>
 <net name="N$18" class="0">
 <segment>
-<wire x1="66.04" y1="99.06" x2="76.2" y2="99.06" width="0.1524" layer="91"/>
-<wire x1="76.2" y1="99.06" x2="76.2" y2="91.44" width="0.1524" layer="91"/>
-<wire x1="76.2" y1="91.44" x2="78.74" y2="91.44" width="0.1524" layer="91"/>
+<wire x1="66.04" y1="99.06" x2="86.36" y2="99.06" width="0.1524" layer="91"/>
+<wire x1="86.36" y1="99.06" x2="86.36" y2="91.44" width="0.1524" layer="91"/>
+<wire x1="86.36" y1="91.44" x2="96.52" y2="91.44" width="0.1524" layer="91"/>
 <pinref part="U1" gate="G$1" pin="*D9"/>
 <pinref part="JP4" gate="G$1" pin="2"/>
@@
 <net name="N$30" class="0">
 <segment>
-<wire x1="66.04" y1="96.52" x2="73.66" y2="96.52" width="0.1524" layer="91"/>
-<wire x1="73.66" y1="96.52" x2="73.66" y2="88.9" width="0.1524" layer="91"/>
-<wire x1="73.66" y1="88.9" x2="78.74" y2="88.9" width="0.1524" layer="91"/>
+<wire x1="66.04" y1="96.52" x2="83.82" y2="96.52" width="0.1524" layer="91"/>
+<wire x1="83.82" y1="96.52" x2="83.82" y2="88.9" width="0.1524" layer="91"/>
 <pinref part="U1" gate="G$1" pin="*D10"/>
 <pinref part="JP4" gate="G$1" pin="3"/>
+<wire x1="83.82" y1="88.9" x2="96.52" y2="88.9" width="0.1524" layer="91"/>
 </segment>
 </net>
 <net name="N$43" class="0">
 <segment>
-<wire x1="66.04" y1="93.98" x2="71.12" y2="93.98" width="0.1524" layer="91"/>
-<wire x1="71.12" y1="93.98" x2="71.12" y2="86.36" width="0.1524" layer="91"/>
-<wire x1="71.12" y1="86.36" x2="78.74" y2="86.36" width="0.1524" layer="91"/>
+<wire x1="66.04" y1="93.98" x2="81.28" y2="93.98" width="0.1524" layer="91"/>
+<wire x1="81.28" y1="93.98" x2="81.28" y2="86.36" width="0.1524" layer="91"/>
+<wire x1="81.28" y1="86.36" x2="96.52" y2="86.36" width="0.1524" layer="91"/>
 <pinref part="U1" gate="G$1" pin="*D11"/>
 <pinref part="JP4" gate="G$1" pin="4"/>
@@
 <net name="N$55" class="0">
 <segment>
-<wire x1="66.04" y1="91.44" x2="68.58" y2="91.44" width="0.1524" layer="91"/>
-<wire x1="68.58" y1="91.44" x2="68.58" y2="83.82" width="0.1524" layer="91"/>
-<wire x1="68.58" y1="83.82" x2="78.74" y2="83.82" width="0.1524" layer="91"/>
+<wire x1="66.04" y1="91.44" x2="78.74" y2="91.44" width="0.1524" layer="91"/>
+<wire x1="78.74" y1="91.44" x2="78.74" y2="83.82" width="0.1524" layer="91"/>
+<wire x1="78.74" y1="83.82" x2="96.52" y2="83.82" width="0.1524" layer="91"/>
 <pinref part="U1" gate="G$1" pin="D12"/>
 <pinref part="JP4" gate="G$1" pin="5"/>
-</segment>
-</net>
-<net name="N$67" class="0">
-<segment>
-<wire x1="78.74" y1="81.28" x2="66.04" y2="81.28" width="0.1524" layer="91"/>
-<wire x1="66.04" y1="81.28" x2="66.04" y2="83.82" width="0.1524" layer="91"/>
-<pinref part="JP4" gate="G$1" pin="6"/>
-<pinref part="U1" gate="G$1" pin="D13"/>
-<pinref part="U1" gate="G$1" pin="SDA"/>
-<wire x1="66.04" y1="83.82" x2="66.04" y2="86.36" width="0.1524" layer="91"/>
-<wire x1="66.04" y1="86.36" x2="66.04" y2="88.9" width="0.1524" layer="91"/>
-<junction x="66.04" y="86.36"/>
-<pinref part="U1" gate="G$1" pin="SCL"/>
-<junction x="66.04" y="83.82"/>
 </segment>
 </net>
@@
 </segment>
 </net>
+<net name="N$3" class="0">
+<segment>
+<pinref part="U1" gate="G$1" pin="D13"/>
+<wire x1="66.04" y1="88.9" x2="76.2" y2="88.9" width="0.1524" layer="91"/>
+<wire x1="76.2" y1="88.9" x2="76.2" y2="81.28" width="0.1524" layer="91"/>
+<pinref part="JP4" gate="G$1" pin="6"/>
+<wire x1="76.2" y1="81.28" x2="96.52" y2="81.28" width="0.1524" layer="91"/>
+</segment>
+</net>
+<net name="N$6" class="0">
+<segment>
+<pinref part="U1" gate="G$1" pin="SDA"/>
+<wire x1="66.04" y1="86.36" x2="73.66" y2="86.36" width="0.1524" layer="91"/>
+<wire x1="73.66" y1="86.36" x2="73.66" y2="73.66" width="0.1524" layer="91"/>
+<pinref part="JP4" gate="G$1" pin="9"/>
+<wire x1="73.66" y1="73.66" x2="96.52" y2="73.66" width="0.1524" layer="91"/>
+</segment>
+</net>
+<net name="N$7" class="0">
+<segment>
+<pinref part="U1" gate="G$1" pin="SCL"/>
+<wire x1="66.04" y1="83.82" x2="71.12" y2="83.82" width="0.1524" layer="91"/>
+<wire x1="71.12" y1="83.82" x2="71.12" y2="71.12" width="0.1524" layer="91"/>
+<pinref part="JP4" gate="G$1" pin="10"/>
+<wire x1="71.12" y1="71.12" x2="96.52" y2="71.12" width="0.1524" layer="91"/>
+</segment>
+</net>
+<net name="AREF" class="0">
+<segment>
+<pinref part="U1" gate="G$1" pin="AREF"/>
+<wire x1="40.64" y1="91.44" x2="38.1" y2="91.44" width="0.1524" layer="91"/>
+<label x="38.1" y="91.44" size="1.27" layer="95" rot="R180" xref="yes"/>
+</segment>
+<segment>
+<pinref part="JP4" gate="G$1" pin="8"/>
+<wire x1="96.52" y1="76.2" x2="91.44" y2="76.2" width="0.1524" layer="91"/>
+<label x="91.44" y="76.2" size="1.27" layer="95" rot="R180" xref="yes"/>
+</segment>
+</net>
